Commit message: feat: viewer, docs, tests, Pi tray / strap slots / camera posts, Makefile pipeline
Claude-Session: https://claude.ai/code/session_017ymwZjQSZTBp7sW4ypCZLL

File: sim/robot/humanoid.urdf (robot description, URDF)
Before this commit: robot humanoid, 21 links, 20 joints
Links:
- link base_link: mass 1.0755 -> 1.0858; geometry visual mesh filename=ads1115_fsr.stl scale=0.001 0.001 0.001; visual mesh filename=battery_3S.stl scale=0.001 0.001 0.001
- link neck_pitch_link: mass 0.1342 -> 0.1343
